Commit message: rename package to ciel_bot

File: catkin_ws/src/ciel_bot/urdf/ciel_bot.xacro (robot description, xacro)
@@ -1,5 +1,5 @@
 <?xml version='1.0'?>
-<robot name="udacity_bot" xmlns:xacro="http://www.ros.org/wiki/xacro">
-    <xacro:include filename="$(find udacity_bot)/urdf/udacity_bot.gazebo" />
+<robot name="ciel_bot" xmlns:xacro="http://www.ros.org/wiki/xacro">
+    <xacro:include filename="$(find ciel_bot)/urdf/ciel_bot.gazebo" />
     <link name="robot_footprint"></link>
     <joint name="robot_footprint_joint" type="fixed">
@@ -22,5 +22,5 @@
             <origin xyz="0 0 0" rpy=" 0 0 0"/>
             <geometry>
-                <box size=".4 .2 .1"/>
+                <cylinder radius="0.2" length="0.15"/>
             </geometry>
         </collision>
@@ -28,9 +28,12 @@
             <origin xyz="0 0 0" rpy=" 0 0 0"/>
             <geometry>
-                <box size=".4 .2 .1"/>
+                <cylinder radius="0.2" length="0.15"/>
             </geometry>
+            <material name="purple">
+                <color rgba="0.5 0 0.5 1"/>
+            </material>
         </visual>
         <collision name='back_caster_collision'>
-            <origin xyz="-0.15 0 -0.05" rpy=" 0 0 0"/>
+            <origin xyz="-0.15 0 -0.1" rpy=" 0 0 0"/>
             <geometry>
                 <sphere radius="0.0499"/>
@@ -38,5 +41,5 @@
         </collision>
         <visual name='back_caster_visual'>
-            <origin xyz="-0.15 0 -0.05" rpy=" 0 0 0"/>
+            <origin xyz="-0.15 0 -0.1" rpy=" 0 0 0"/>
             <geometry>
                 <sphere radius="0.05"/>
@@ -44,5 +47,5 @@
         </visual>
         <collision name='front_caster_collision'>
-            <origin xyz="0.15 0 -0.05" rpy=" 0 0 0"/>
+            <origin xyz="0.15 0 -0.1" rpy=" 0 0 0"/>
             <geometry>
                 <sphere radius="0.0499"/>
@@ -50,5 +53,5 @@
         </collision>
         <visual name='front_caster_visual'>
-            <origin xyz="0.15 0 -0.05" rpy=" 0 0 0"/>
+            <origin xyz="0.15 0 -0.1" rpy=" 0 0 0"/>
             <geometry>
                 <sphere radius="0.05"/>
@@ -58,5 +61,5 @@
     <!-- *********  Left Wheel ******************************** -->
     <joint name="left_wheel_hinge" type="continuous">
-        <origin xyz="0 0.15 0" rpy="0 0 0"/>
+        <origin xyz="0 0.2 -0.05" rpy="0 0 0"/>
         <child link="left_wheel"/>
         <parent link="chassis"/>
@@ -80,6 +83,6 @@
             </geometry>
             <origin xyz="0 0 0" rpy="0 1.5707 1.5707"/>
-            <material name="white">
-                <color rgba="1 1 1 1"/>
+            <material name="green">
+                <color rgba="0 1 0 1"/>
             </material>
         </visual>
@@ -93,5 +96,5 @@
     <!-- *********  Right Wheel ******************************** -->
     <joint name="right_wheel_hinge" type="continuous">
-        <origin xyz="0 -0.15 0" rpy="0 0 0"/>
+        <origin xyz="0 -0.2 -0.05" rpy="0 0 0"/>
         <child link="right_wheel"/>
         <parent link="chassis"/>
@@ -115,6 +118,6 @@
             </geometry>
             <origin xyz="0 0 0" rpy="0 1.5707 1.5707"/>
-            <material name="white">
-                <color rgba="1 1 1 1"/>
+            <material name="green">
+                <color rgba="0 1 0 1"/>
             </material>
         </visual>
@@ -128,5 +131,5 @@
     <!-- *********  Camera ******************************** -->
     <joint name="camera_joint" type="fixed">
-        <origin xyz="0.25 0 0" rpy="0 0 0"/>
+        <origin xyz="0.0 0 0" rpy="0 0 0"/>
         <child link="camera"/>
         <parent link="chassis"/>
@@ -160,5 +163,5 @@
     <!-- *********  Laser Rangefinder ******************************** -->
     <joint type="fixed" name="hokuyo_joint">
-        <origin xyz="0.15 0 0.1" rpy="0 0 0"/>
+        <origin xyz="0.0 0 0.1" rpy="0 0 0"/>
         <child link="hokuyo"/>
         <parent link="chassis"/>
@@ -176,5 +179,5 @@
         <visual>
             <geometry>
-                <mesh filename="package://udacity_bot/meshes/hokuyo.dae"/>
+                <mesh filename="package://ciel_bot/meshes/hokuyo.dae"/>
             </geometry>
             <origin xyz="0 0 0" rpy="0 0 0"/>

Commit message: fixing up bot, launch world variable, READMe

File: catkin_ws/src/ciel_bot/urdf/ciel_bot.xacro (robot description, xacro)
@@ -4,10 +4,10 @@
     <link name="robot_footprint"></link>
     <joint name="robot_footprint_joint" type="fixed">
-        <origin xyz="0 0 0" rpy="0 0 0" />
+        <origin xyz="0 0.1 0" rpy="0 0 0" />
         <parent link="robot_footprint"/>
         <child link="chassis" />
     </joint>
     <link name='chassis'>
-        <pose>0 0 0.1 0 0 0</pose>
+        <pose>0 0 0.0 0 0 0</pose>
         <inertial>
             <mass value="15.0"/>
@@ -131,5 +131,5 @@
     <!-- *********  Camera ******************************** -->
     <joint name="camera_joint" type="fixed">
-        <origin xyz="0.0 0 0" rpy="0 0 0"/>
+        <origin xyz="0.2 0 0" rpy="0 0 0"/>
         <child link="camera"/>
         <parent link="chassis"/>
@@ -163,5 +163,5 @@
     <!-- *********  Laser Rangefinder ******************************** -->
     <joint type="fixed" name="hokuyo_joint">
-        <origin xyz="0.0 0 0.1" rpy="0 0 0"/>
+        <origin xyz="0 0 0.1" rpy="0 0 0"/>
         <child link="hokuyo"/>
         <parent link="chassis"/>

Commit message: Fix rgbd gazebo fram

File: catkin_ws/src/ciel_bot/urdf/ciel_bot.xacro (robot description, xacro)
@@ -130,13 +130,8 @@
     </link>
     <!-- *********  Camera ******************************** -->
-    <joint name="camera_joint" type="fixed">
-        <origin xyz="0.2 0 0" rpy="0 0 0"/>
-        <child link="camera"/>
-        <parent link="chassis"/>
-    </joint>
-    <link name='camera'>
+    <link name="camera">
         <inertial>
             <mass value="0.1"/>
-            <origin xyz="0 0 0" rpy="0 0 0"/>
+            <origin xyz="0.0 0 0" rpy=" 0 0 0"/>
             <inertia
                     ixx="1e-6" ixy="0" ixz="0"
@@ -145,20 +140,31 @@
             />
         </inertial>
-        <visual>
+        <collision name='collision'>
+            <origin xyz="0.0 0 0" rpy=" 0 0 0"/>
             <geometry>
                 <box size="0.05 0.05 0.05"/>
             </geometry>
-            <origin xyz="0 0 0" rpy="0 0 0"/>
-            <material name="blue">
-                <color rgba="0 0 1 1"/>
-            </material>
-        </visual>
-        <collision>
+        </collision>
+        <visual name='camera_visual'>
+            <origin xyz="0.0 0 0" rpy=" 0 0 0"/>
             <geometry>
                 <box size="0.05 0.05 0.05"/>
             </geometry>
-            <origin xyz="0 0 0" rpy="0 0 0"/>
-        </collision>
+        </visual>
     </link>
+    <joint type="fixed" name="camera_joint">
+        <origin xyz="0.2 0 0" rpy="0 0 0"/>
+        <child link="camera"/>
+        <parent link="chassis"/>
+        <axis xyz="0 1 0" rpy="0 0 0"/>
+        <limit effort="10000" velocity="1000"/>
+        <dynamics damping="1.0" friction="1.0"/>
+    </joint>
+    <link name="camera_rgbd_frame"></link>
+    <joint name="camera_rgbd_joint" type="fixed">
+        <origin xyz="0 0 0" rpy="-${pi/2} 0 -${pi/2}"/>
+        <parent link="camera"/>
+        <child link="camera_rgbd_frame"/>
+    </joint>
     <!-- *********  Laser Rangefinder ******************************** -->
     <joint type="fixed" name="hokuyo_joint">
